File: washear.sch (KiCad schematic (older format))
At the start: 12 parts

Commit message: Complete the draft schematics
Parts:
- removed U?: LM324, symbol LM324
- added C?: C, ~, symbol C
- added D?: LED, ~, symbol LED
- added Q?: PNP, ~, symbol PNP
- added R? (x2): 1M, ~, symbol R
- added R? (x5): R, ~, symbol R
- added RV?: 2k2, ~, symbol POT
- added SW?: OFF, ~, symbol SW_PUSH
- added SW?: ON, ~, symbol SW_PUSH
- added U? (x2): TLC27L2, symbol TLC27L2
- added U?: TLC555, symbol TLC555
Connections:
- wire segments 24 -> 61
Other:
- moved on the sheet: R?, RV?, U?A, U?B

Commit message: Complete second draft schematics
Parts:
- removed C?: CP1, ~, symbol CP1
- removed C?: C, ~, symbol C
- removed D?: LED, ~, symbol LED
- removed R? (x6): 1M, ~, symbol R
- removed R? (x6): R, ~, symbol R
- removed U?: TLC555, symbol TLC555
- added C?: 0.1uF, symbol C
- added C? (x2): CP, symbol CP
- added D?: LED, symbol LED
- added R? (x6): R, symbol R
- added R? (x6): 1M, symbol R
- added U?: TLC555, ~, symbol TLC555
- added U?: 74HC02, ~, symbol 74HC02
Connections:
- net labels added: GND, VDD
- wire segments 61 -> 60
Other:
- moved on the sheet: RV?, SW?, U?A, U?B

Commit message: Capture first complete working schematic
Parts:
- removed D?: DIODE, ~, symbol DIODE
- removed Q?: PNP, ~, symbol PNP
- removed R?: R, symbol R
- removed U?: TLC555, ~, symbol TLC555
- added C?: 0.1uF, symbol C
- added D? (x2): 1N4005, symbol D
- added Q?: 2n2222a, symbol Q_NPN_EBC
- added R?: 1K, symbol R
- added R?: 10K, symbol R
- added U?: TLC555, symbol TLC555
- C?: value CP -> 2.2uF
- C?: value CP -> 22uF
- D?: value LED -> 1.8V 20mA
- R?: value R -> 12K
- R? (x2): value R -> 1M
- R?: value R -> 100K
- R?: value R -> 220
- RV?: value 2k2 -> 200K
- RV?: value 2k2 -> 1M
Connections:
- net labels added: +5V
- net labels removed: VDD
- wire segments 60 -> 103
Other:
- moved on the sheet: C?, D?, R?, RV?, SW?, U?A, U?B, U?C
